File: base_convert_bin.sch (KiCad schematic (older format))
At the start: 36 parts, among them Q18 Q_PNP_BEC, Q19 Q_PNP_BEC, Q20 Q_PNP_BEC, Q21 Q_PNP_BEC, Q22 Q_NPN_BEC, Q23 Q_NPN_BEC, Q24 Q_NPN_BEC, Q25 Q_NPN_BEC

Commit message: updated shema fields. Raplced tack switch with 4 pin footprint
Using 4 pin tack switch to ease pcb layout connecitions. Also updated component fields in schema
Parts:
- D1, D10, D11, D12, D13, D14, D15, D16, D2, D3, D4, D5, D6, D7, D8, D9, R26, R27, R28, R29, R30, R31, R32, R33, R34, R35, R36, R37: Description NONE -> (none); Manufacture NONE -> (none); Mfg Part Number NONE -> (none); Package NONE -> (none)
- Q18: Description (none) -> TRANS PNP 40V 0.2A SOT23; Manufacture (none) -> Nexperia USA Inc.; Mfg Part Number (none) -> PMBT3906,235; Package (none) -> SOT-23
- Q19: Description (none) -> TRANS PNP 40V 0.2A SOT24; Manufacture (none) -> Nexperia USA Inc.; Mfg Part Number (none) -> PMBT3906,236; Package (none) -> SOT-23
- Q20: Description (none) -> TRANS PNP 40V 0.2A SOT26; Manufacture (none) -> Nexperia USA Inc.; Mfg Part Number (none) -> PMBT3906,238; Package (none) -> SOT-23
- Q21: Description (none) -> TRANS PNP 40V 0.2A SOT27; Manufacture (none) -> Nexperia USA Inc.; Mfg Part Number (none) -> PMBT3906,239; Package (none) -> SOT-23
- Q22, Q23, Q24, Q25: Description (none) -> TRANSISTOR, NPN, 40V, 0.2A, 100A; Manufacture (none) -> Taiwan Semiconductor Corporation; Mfg Part Number (none) -> MMBT3904L RFG; Package (none) -> SOT-23
