File: base_convert_display.sch (KiCad schematic (older format))
At the start: 49 parts, among them Q10 Q_PNP_BEC, Q11 Q_NPN_BEC, Q12 Q_NPN_BEC, Q13 Q_NPN_BEC, Q14 Q_NPN_BEC, Q15 Q_NPN_BEC, Q16 Q_NPN_BEC, Q17 Q_NPN_BEC, Q2 Q_PNP_BEC, Q26 Q_PNP_BEC, Q27 Q_NPN_BEC, Q3 Q_PNP_BEC, Q4 Q_PNP_BEC, Q5 Q_PNP_BEC, Q6 Q_PNP_BEC, Q7 Q_PNP_BEC, Q8 Q_PNP_BEC, Q9 Q_PNP_BEC

Commit message: Push and shove for the win!
To Do: clean up.
Connections:
- net DEC1: no longer R7.2
- net DEC2: no longer R8.2
- net DEC3: no longer R9.2
- net DEC4: no longer R10.2
- net DEC5: no longer R11.2
- net DEC6: no longer R38.2
- net HEX1: no longer R3.2
- net HEX2: no longer R4.2
- net HEX3: no longer R5.2
- net HEX4: no longer R6.2
- new net ~DEC1: R7.2
- new net ~DEC2: R8.2
- new net ~DEC3: R9.2
- new net ~DEC4: R10.2
- new net ~DEC5: R11.2
- new net ~DEC6: R38.2
- new net ~HEX1: R3.2
- new net ~HEX2: R4.2
- new net ~HEX3: R5.2
- new net ~HEX4: R6.2
Changed lines of the file:
@@
 LIBS:MSP430
 LIBS:Switch_CK
+LIBS:Switch_Generic
 LIBS:base_convert-cache
 LIBS:4xxx
@@
 $EndComp
 $Comp
-L VCC #PWR11
+L VCC #PWR011
 U 1 1 5AEAC3DE
 P 1750 700
-F 0 "#PWR11" H 1750 550 50  0001 C CNN
+F 0 "#PWR011" H 1750 550 50  0001 C CNN
 F 1 "VCC" H 1750 850 50  0000 C CNN
 F 2 "" H 1750 700 50  0001 C CNN
@@
 $EndComp
 $Comp
-L VCC #PWR12
+L VCC #PWR012
 U 1 1 5AEAC963
 P 1750 1400
-F 0 "#PWR12" H 1750 1250 50  0001 C CNN
+F 0 "#PWR012" H 1750 1250 50  0001 C CNN
 F 1 "VCC" H 1750 1550 50  0000 C CNN
 F 2 "" H 1750 1400 50  0001 C CNN
@@
 $EndComp
 $Comp
-L VCC #PWR13
+L VCC #PWR013
 U 1 1 5AEACAA1
 P 1750 2100
-F 0 "#PWR13" H 1750 1950 50  0001 C CNN
+F 0 "#PWR013" H 1750 1950 50  0001 C CNN
 F 1 "VCC" H 1750 2250 50  0000 C CNN
 F 2 "" H 1750 2100 50  0001 C CNN
@@
 $EndComp
 $Comp
-L VCC #PWR14
+L VCC #PWR014
 U 1 1 5AEACAB9
 P 1750 2800
-F 0 "#PWR14" H 1750 2650 50  0001 C CNN
+F 0 "#PWR014" H 1750 2650 50  0001 C CNN
 F 1 "VCC" H 1750 2950 50  0000 C CNN
 F 2 "" H 1750 2800 50  0001 C CNN
@@
 $EndComp
 $Comp
-L VCC #PWR15
+L VCC #PWR015
 U 1 1 5AEB118F
 P 1750 3500
-F 0 "#PWR15" H 1750 3350 50  0001 C CNN
+F 0 "#PWR015" H 1750 3350 50  0001 C CNN
 F 1 "VCC" H 1750 3650 50  0000 C CNN
 F 2 "" H 1750 3500 50  0001 C CNN
@@
 $EndComp
 $Comp
-L VCC #PWR16
+L VCC #PWR016
 U 1 1 5AEB11A9
 P 1750 4200
-F 0 "#PWR16" H 1750 4050 50  0001 C CNN
+F 0 "#PWR016" H 1750 4050 50  0001 C CNN
 F 1 "VCC" H 1750 4350 50  0000 C CNN
 F 2 "" H 1750 4200 50  0001 C CNN
@@
 $EndComp
 $Comp
-L VCC #PWR17
+L VCC #PWR017
 U 1 1 5AEB11C3
 P 1750 4900
-F 0 "#PWR17" H 1750 4750 50  0001 C CNN
+F 0 "#PWR017" H 1750 4750 50  0001 C CNN
 F 1 "VCC" H 1750 5050 50  0000 C CNN
 F 2 "" H 1750 4900 50  0001 C CNN
@@
 $EndComp
 $Comp
-L VCC #PWR18
+L VCC #PWR018
 U 1 1 5AEB11DD
 P 1750 5600
-F 0 "#PWR18" H 1750 5450 50  0001 C CNN
+F 0 "#PWR018" H 1750 5450 50  0001 C CNN
 F 1 "VCC" H 1750 5750 50  0000 C CNN
 F 2 "" H 1750 5600 50  0001 C CNN
@@
 $EndComp
 $Comp
-L VCC #PWR19
+L VCC #PWR019
 U 1 1 5AEB1797
 P 1750 6300
-F 0 "#PWR19" H 1750 6150 50  0001 C CNN
+F 0 "#PWR019" H 1750 6150 50  0001 C CNN
 F 1 "VCC" H 1750 6450 50  0000 C CNN
 F 2 "" H 1750 6300 50  0001 C CNN
@@
 $EndComp
 $Comp
-L GND #PWR21
+L GND #PWR020
 U 1 1 5AEB7854
 P 9000 1250
-F 0 "#PWR21" H 9000 1000 50  0001 C CNN
+F 0 "#PWR020" H 9000 1000 50  0001 C CNN
 F 1 "GND" H 9000 1100 50  0000 C CNN
 F 2 "" H 9000 1250 50  0001 C CNN
@@
 $EndComp
 $Comp
-L GND #PWR22
+L GND #PWR021
 U 1 1 5AEB9888
 P 9000 2050
-F 0 "#PWR22" H 9000 1800 50  0001 C CNN
+F 0 "#PWR021" H 9000 1800 50  0001 C CNN
 F 1 "GND" H 9000 1900 50  0000 C CNN
 F 2 "" H 9000 2050 50  0001 C CNN
@@
 $EndComp
 $Comp
-L GND #PWR23
+L GND #PWR022
 U 1 1 5AEB9B0D
 P 9000 2850
-F 0 "#PWR23" H 9000 2600 50  0001 C CNN
+F 0 "#PWR022" H 9000 2600 50  0001 C CNN
 F 1 "GND" H 9000 2700 50  0000 C CNN
 F 2 "" H 9000 2850 50  0001 C CNN
@@
 $EndComp
 $Comp
-L GND #PWR24
+L GND #PWR023
 U 1 1 5AEB9B31
 P 9000 3650
-F 0 "#PWR24" H 9000 3400 50  0001 C CNN
+F 0 "#PWR023" H 9000 3400 50  0001 C CNN
 F 1 "GND" H 9000 3500 50  0000 C CNN
 F 2 "" H 9000 3650 50  0001 C CNN
@@
 $EndComp
 $Comp
-L GND #PWR25
+L GND #PWR024
 U 1 1 5AEB9F7B
 P 9000 4450
-F 0 "#PWR25" H 9000 4200 50  0001 C CNN
+F 0 "#PWR024" H 9000 4200 50  0001 C CNN
 F 1 "GND" H 9000 4300 50  0000 C CNN
 F 2 "" H 9000 4450 50  0001 C CNN
@@
 $EndComp
 $Comp
-L GND #PWR26
+L GND #PWR025
 U 1 1 5AEB9F9F
 P 9000 5250
-F 0 "#PWR26" H 9000 5000 50  0001 C CNN
+F 0 "#PWR025" H 9000 5000 50  0001 C CNN
 F 1 "GND" H 9000 5100 50  0000 C CNN
 F 2 "" H 9000 5250 50  0001 C CNN
@@
 $EndComp
 $Comp
-L GND #PWR27
+L GND #PWR026
 U 1 1 5AEB9FC3
 P 9000 6050
-F 0 "#PWR27" H 9000 5800 50  0001 C CNN
+F 0 "#PWR026" H 9000 5800 50  0001 C CNN
 F 1 "GND" H 9000 5900 50  0000 C CNN
 F 2 "" H 9000 6050 50  0001 C CNN
@@
 $EndComp
 $Comp
-L VCC #PWR20
+L VCC #PWR027
 U 1 1 5AF53099
 P 1750 7000
-F 0 "#PWR20" H 1750 6850 50  0001 C CNN
+F 0 "#PWR027" H 1750 6850 50  0001 C CNN
 F 1 "VCC" H 1750 7150 50  0000 C CNN
 F 2 "" H 1750 7000 50  0001 C CNN
@@
 $EndComp
 $Comp
-L GND #PWR28
+L GND #PWR028
 U 1 1 5AF5696E
 P 9000 6850
-F 0 "#PWR28" H 9000 6600 50  0001 C CNN
+F 0 "#PWR028" H 9000 6600 50  0001 C CNN
 F 1 "GND" H 9000 6700 50  0000 C CNN
 F 2 "" H 9000 6850 50  0001 C CNN
@@
 G
 Text HLabel 1100 950  0    60   Input ~ 0
-HEX1
+~HEX1
 Text HLabel 1100 1650 0    60   Input ~ 0
-HEX2
+~HEX2
 Text HLabel 1100 2350 0    60   Input ~ 0
-HEX3
+~HEX3
 Text HLabel 1100 3050 0    60   Input ~ 0
-HEX4
+~HEX4
 Text HLabel 1100 3750 0    60   Input ~ 0
-DEC1
+~DEC1
 Text HLabel 1100 4450 0    60   Input ~ 0
-DEC2
+~DEC2
 Text HLabel 1100 5150 0    60   Input ~ 0
-DEC3
+~DEC3
 Text HLabel 1100 5850 0    60   Input ~ 0
-DEC4
+~DEC4
 Text HLabel 1100 6550 0    60   Input ~ 0
-DEC5
+~DEC5
 Text HLabel 9700 1000 2    60   Input ~ 0
 SEG-A
@@
 DEC6
 Text HLabel 1100 7250 0    60   Input ~ 0
-DEC6
+~DEC6
 Text Label 4100 5100 0    60   ~ 0
 DEC6
