File: base_convert_keypad.sch (KiCad schematic (older format))
At the start: 17 parts, among them SW1 CLEAR, SW19 0, SW20 4, SW21 8, SW22 C, SW23 1, SW24 5, SW25 9, SW26 D, SW27 2, SW28 6, SW29 A, SW30 E, SW31 3, SW32 7, SW33 B, SW34 F

Commit message: component selection update
Parts:
- SW1: Package 6mm SMT -> SMT
- SW19, SW20, SW21, SW22, SW23, SW24, SW25, SW26, SW27, SW28, SW29, SW30, SW31, SW32, SW33, SW34: footprint Buttons_Switches_THT:SW_TH_Tactile_Omron_B3F-10xx -> (none); Package 6mm SMT -> SMT

Commit message: update keypad switch footprint to smd
Parts:
- SW1, SW19, SW20, SW21, SW22, SW23, SW24, SW25, SW26, SW27, SW28, SW29, SW30, SW31, SW32, SW33, SW34: footprint (none) -> Switch_CK:CK_PTS645_6mm_SMD
Changed lines of the file:
@@
 F 0 "SW20" H 5700 3100 50  0000 L CNN
 F 1 "4" H 5650 2750 50  0000 C CNN
-F 2 "" H 5650 3200 50  0001 C CNN
+F 2 "Switch_CK:CK_PTS645_6mm_SMD" H 5650 3200 50  0001 C CNN
 F 3 "https://www.ckswitches.com/media/1471/pts645.pdf" H 5650 3200 50  0001 C CNN
 F 4 "SWITCH TACTILE SPST-NO 0.05A 12V" H 5650 3000 60  0001 C CNN "Description"
@@
 F 0 "SW24" H 4900 3100 50  0000 L CNN
 F 1 "5" H 4850 2750 50  0000 C CNN
-F 2 "" H 4850 3200 50  0001 C CNN
+F 2 "Switch_CK:CK_PTS645_6mm_SMD" H 4850 3200 50  0001 C CNN
 F 3 "https://www.ckswitches.com/media/1471/pts645.pdf" H 4850 3200 50  0001 C CNN
 F 4 "SWITCH TACTILE SPST-NO 0.05A 12V" H 4850 3000 60  0001 C CNN "Description"
@@
 F 0 "SW28" H 4100 3100 50  0000 L CNN
 F 1 "6" H 4050 2750 50  0000 C CNN
-F 2 "" H 4050 3200 50  0001 C CNN
+F 2 "Switch_CK:CK_PTS645_6mm_SMD" H 4050 3200 50  0001 C CNN
 F 3 "https://www.ckswitches.com/media/1471/pts645.pdf" H 4050 3200 50  0001 C CNN
 F 4 "SWITCH TACTILE SPST-NO 0.05A 12V" H 4050 3000 60  0001 C CNN "Description"
@@
 F 0 "SW22" H 6500 3100 50  0000 L CNN
 F 1 "C" H 6450 2750 50  0000 C CNN
-F 2 "" H 6450 3200 50  0001 C CNN
+F 2 "Switch_CK:CK_PTS645_6mm_SMD" H 6450 3200 50  0001 C CNN
 F 3 "https://www.ckswitches.com/media/1471/pts645.pdf" H 6450 3200 50  0001 C CNN
 F 4 "SWITCH TACTILE SPST-NO 0.05A 12V" H 6450 3000 60  0001 C CNN "Description"
@@
 F 0 "SW33" H 6500 2450 50  0000 L CNN
 F 1 "B" H 6450 2100 50  0000 C CNN
-F 2 "" H 6450 2550 50  0001 C CNN
+F 2 "Switch_CK:CK_PTS645_6mm_SMD" H 6450 2550 50  0001 C CNN
 F 3 "https://www.ckswitches.com/media/1471/pts645.pdf" H 6450 2550 50  0001 C CNN
 F 4 "SWITCH TACTILE SPST-NO 0.05A 12V" H 6450 2350 60  0001 C CNN "Description"
@@
 F 0 "SW23" H 5700 2450 50  0000 L CNN
 F 1 "1" H 5650 2100 50  0000 C CNN
-F 2 "" H 5650 2550 50  0001 C CNN
+F 2 "Switch_CK:CK_PTS645_6mm_SMD" H 5650 2550 50  0001 C CNN
 F 3 "https://www.ckswitches.com/media/1471/pts645.pdf" H 5650 2550 50  0001 C CNN
 F 4 "SWITCH TACTILE SPST-NO 0.05A 12V" H 5650 2350 60  0001 C CNN "Description"
@@
 F 0 "SW27" H 4900 2450 50  0000 L CNN
 F 1 "2" H 4850 2100 50  0000 C CNN
-F 2 "" H 4850 2550 50  0001 C CNN
+F 2 "Switch_CK:CK_PTS645_6mm_SMD" H 4850 2550 50  0001 C CNN
 F 3 "https://www.ckswitches.com/media/1471/pts645.pdf" H 4850 2550 50  0001 C CNN
 F 4 "SWITCH TACTILE SPST-NO 0.05A 12V" H 4850 2350 60  0001 C CNN "Description"
@@
 F 0 "SW31" H 4100 2450 50  0000 L CNN
 F 1 "3" H 4050 2100 50  0000 C CNN
-F 2 "" H 4050 2550 50  0001 C CNN
+F 2 "Switch_CK:CK_PTS645_6mm_SMD" H 4050 2550 50  0001 C CNN
 F 3 "https://www.ckswitches.com/media/1471/pts645.pdf" H 4050 2550 50  0001 C CNN
 F 4 "SWITCH TACTILE SPST-NO 0.05A 12V" H 4050 2350 60  0001 C CNN "Description"
@@
 F 0 "SW19" H 4900 4400 50  0000 L CNN
 F 1 "0" H 4850 4050 50  0000 C CNN
-F 2 "" H 4850 4500 50  0001 C CNN
+F 2 "Switch_CK:CK_PTS645_6mm_SMD" H 4850 4500 50  0001 C CNN
 F 3 "https://www.ckswitches.com/media/1471/pts645.pdf" H 4850 4500 50  0001 C CNN
 F 4 "SWITCH TACTILE SPST-NO 0.05A 12V" H 4850 4300 60  0001 C CNN "Description"
@@
 F 0 "SW29" H 5700 4400 50  0000 L CNN
 F 1 "A" H 5650 4050 50  0000 C CNN
-F 2 "" H 5650 4500 50  0001 C CNN
+F 2 "Switch_CK:CK_PTS645_6mm_SMD" H 5650 4500 50  0001 C CNN
 F 3 "https://www.ckswitches.com/media/1471/pts645.pdf" H 5650 4500 50  0001 C CNN
 F 4 "SWITCH TACTILE SPST-NO 0.05A 12V" H 5650 4300 60  0001 C CNN "Description"
@@
 F 0 "SW30" H 6500 4400 50  0000 L CNN
 F 1 "E" H 6450 4050 50  0000 C CNN
-F 2 "" H 6450 4500 50  0001 C CNN
+F 2 "Switch_CK:CK_PTS645_6mm_SMD" H 6450 4500 50  0001 C CNN
 F 3 "https://www.ckswitches.com/media/1471/pts645.pdf" H 6450 4500 50  0001 C CNN
 F 4 "SWITCH TACTILE SPST-NO 0.05A 12V" H 6450 4300 60  0001 C CNN "Description"
@@
 F 0 "SW34" H 4100 4400 50  0000 L CNN
 F 1 "F" H 4050 4050 50  0000 C CNN
-F 2 "" H 4050 4500 50  0001 C CNN
+F 2 "Switch_CK:CK_PTS645_6mm_SMD" H 4050 4500 50  0001 C CNN
 F 3 "https://www.ckswitches.com/media/1471/pts645.pdf" H 4050 4500 50  0001 C CNN
 F 4 "SWITCH TACTILE SPST-NO 0.05A 12V" H 4050 4300 60  0001 C CNN "Description"
@@
 F 0 "SW21" H 4900 3750 50  0000 L CNN
 F 1 "8" H 4850 3400 50  0000 C CNN
-F 2 "" H 4850 3850 50  0001 C CNN
+F 2 "Switch_CK:CK_PTS645_6mm_SMD" H 4850 3850 50  0001 C CNN
 F 3 "https://www.ckswitches.com/media/1471/pts645.pdf" H 4850 3850 50  0001 C CNN
 F 4 "SWITCH TACTILE SPST-NO 0.05A 12V" H 4850 3650 60  0001 C CNN "Description"
@@
 F 0 "SW25" H 4100 3750 50  0000 L CNN
 F 1 "9" H 4050 3400 50  0000 C CNN
-F 2 "" H 4050 3850 50  0001 C CNN
+F 2 "Switch_CK:CK_PTS645_6mm_SMD" H 4050 3850 50  0001 C CNN
 F 3 "https://www.ckswitches.com/media/1471/pts645.pdf" H 4050 3850 50  0001 C CNN
 F 4 "SWITCH TACTILE SPST-NO 0.05A 12V" H 4050 3650 60  0001 C CNN "Description"
@@
 F 0 "SW32" H 5700 3750 50  0000 L CNN
 F 1 "7" H 5650 3400 50  0000 C CNN
-F 2 "" H 5650 3850 50  0001 C CNN
+F 2 "Switch_CK:CK_PTS645_6mm_SMD" H 5650 3850 50  0001 C CNN
 F 3 "https://www.ckswitches.com/media/1471/pts645.pdf" H 5650 3850 50  0001 C CNN
 F 4 "SWITCH TACTILE SPST-NO 0.05A 12V" H 5650 3650 60  0001 C CNN "Description"
@@
 F 0 "SW26" H 6500 3750 50  0000 L CNN
 F 1 "D" H 6450 3400 50  0000 C CNN
-F 2 "" H 6450 3850 50  0001 C CNN
+F 2 "Switch_CK:CK_PTS645_6mm_SMD" H 6450 3850 50  0001 C CNN
 F 3 "https://www.ckswitches.com/media/1471/pts645.pdf" H 6450 3850 50  0001 C CNN
 F 4 "SWITCH TACTILE SPST-NO 0.05A 12V" H 6450 3650 60  0001 C CNN "Description"
@@
 F 0 "SW1" H 6500 1800 50  0000 L CNN
 F 1 "CLEAR" H 6450 1450 50  0000 C CNN
-F 2 "" H 6450 1900 50  0001 C CNN
+F 2 "Switch_CK:CK_PTS645_6mm_SMD" H 6450 1900 50  0001 C CNN
 F 3 "https://www.ckswitches.com/media/1471/pts645.pdf" H 6450 1900 50  0001 C CNN
 F 4 "SWITCH TACTILE SPST-NO 0.05A 12V" H 6450 1700 60  0001 C CNN "Description"
